File: pcb/Nu6509_v4.sch (EAGLE design)
At the start: 22 parts, among them IC1 6509, IC3 (C)02/'816, IC4 XC9572XL

Commit message: Switch name to Nu6509
Parts:
- added R2: 10K, rcl:R-US_R0402
Connections:
- net !ABORT: now also R2.2
- net +3V3: now also R2.1
Changed lines of the file:
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@@
 <part name="R1" library="rcl" deviceset="R-US_" device="R0402" value="10K"/>
 <part name="GND12" library="supply1" deviceset="GND" device=""/>
+<part name="R2" library="rcl" deviceset="R-US_" device="R0402" value="10K"/>
+<part name="+3V5" library="supply1" deviceset="+3V3" device=""/>
 </parts>
 <sheets>
@@
 </instance>
 <instance part="GND12" gate="1" x="99.06" y="170.18"/>
+<instance part="R2" gate="G$1" x="91.44" y="180.34" smashed="yes" rot="R270">
+<attribute name="NAME" x="92.9386" y="184.15" size="1.778" layer="95" rot="R270"/>
+<attribute name="VALUE" x="88.138" y="184.15" size="1.778" layer="96" rot="R270"/>
+</instance>
+<instance part="+3V5" gate="G$1" x="91.44" y="190.5"/>
 </instances>
 <busses>
@@
 <pinref part="3V3" gate="G$1" pin="TP"/>
 </segment>
+<segment>
+<pinref part="+3V5" gate="G$1" pin="+3V3"/>
+<pinref part="R2" gate="G$1" pin="1"/>
+<wire x1="91.44" y1="187.96" x2="91.44" y2="185.42" width="0.1524" layer="91"/>
+</segment>
 </net>
 <net name="GND" class="0">
@@
 <label x="223.52" y="55.88" size="1.27" layer="95" rot="R270" xref="yes"/>
 </segment>
-</net>
+<segment>
+<pinref part="R2" gate="G$1" pin="2"/>
+<wire x1="91.44" y1="175.26" x2="91.44" y2="172.72" width="0.1524" layer="91"/>
+<label x="91.44" y="172.72" size="1.27" layer="95" rot="R270" xref="yes"/>
+</segment>
+</net>
